File: Kicad/Camper_Energy_Saver.kicad_sch (KiCad schematic)
At the start: 59 parts, among them J1 IDC_13X2, J2 Conn_01x03_Pin, J3 Conn_01x03_Pin, J4 IDC_5X2, J5 Conn_01x03_Pin, K1 N.M., K2 G5V-1-DC12V, K3 Relay_SPST-NO, Q1 N.M., Q2 BC337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

Commit message: SCHEMA
Parts:
- added R21: 2k2, symbol Device:R
- added R22: 1k, symbol Device:R
Connections:
- net D11: now also R22.1
- net GND: now also R21.2
- new net: R21.1, R22.2
Other:
- note added: "BLUETOOTH"
- note added: "MODULO MAK-NANO2RL"
- note added: "PANNELLI SOLARI"
- moved on the sheet: A1, BT1, BT2, BZ1, C1, C2, C3, C4, C5, C6, D1, D10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
