File: Kicad/Camper_Energy_Saver.kicad_sch (KiCad schematic)
At the start: 59 parts, among them J1 IDC_13X2, J2 Conn_01x03_Pin, J3 Conn_01x03_Pin, J4 IDC_5X2, J5 Conn_01x03_Pin, K1 N.M., K2 G5V-1-DC12V, K4 N.M., Q1 N.M., Q2 BC337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

Commit message: docs
Parts:
- added SW1: DISABILITA, symbol Switch:SW_DPST_x2
Connections:
- net NO1: now also SW1.2 (B)
Other:
- note added: "30"
- note added: "85"
- note added: "86"
- note added: "87"
- note added: "87A"
- note added: "BLUETOOTH HC05"
- note removed: "BLUETOOTH"
Changed lines of the file:
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@@
 		)
 	)
+	(text "30"
+		(exclude_from_sim no)
+		(at 347.472 36.322 90)
+		(effects
+			(font
+				(size 1.27 1.27)
+			)
+		)
+	)
 	(text "V_serv\n"
 		(exclude_from_sim no)
@@
 		)
 	)
+	(text "87"
+		(exclude_from_sim no)
+		(at 341.63 42.926 90)
+		(effects
+			(font
+				(size 1.27 1.27)
+			)
+		)
+	)
 	(text "BLU"
 		(exclude_from_sim no)
@@
 	(text "MODULO MAK-NANO2RL"
 		(exclude_from_sim no)
-		(at 238.252 224.282 0)
+		(at 220.218 223.52 0)
 		(effects
 			(font
-				(size 2.54 2.54)
+				(size 4.572 4.572)
+				(thickness 0.9144)
+				(bold yes)
 			)
 		)
@@
 		)
 	)
+	(text "87A"
+		(exclude_from_sim no)
+		(at 349.25 42.418 90)
+		(effects
+			(font
+				(size 1.27 1.27)
+			)
+		)
+	)
 	(text "SOGLIA BASSA"
 		(exclude_from_sim no)
@@
 		)
 	)
-	(text "BLUETOOTH\n"
+	(text "85"
+		(exclude_from_sim no)
+		(at 334.01 43.18 90)
+		(effects
+			(font
+				(size 1.27 1.27)
+			)
+		)
+	)
+	(text "BLUETOOTH HC05\n"
 		(exclude_from_sim no)
-		(at 132.842 58.42 0)
+		(at 108.204 51.816 0)
 		(effects
 			(font
@@
 		)
 	)
+	(text "86"
+		(exclude_from_sim no)
+		(at 334.01 36.068 90)
+		(effects
+			(font
+				(size 1.27 1.27)
+			)
+		)
+	)
 	(junction
 		(at 340.36 88.9)
@@
 	(wire
 		(pts
-			(xy 335.28 31.75) (xy 311.15 31.75)
-		)
-		(stroke
-			(width 0)
-			(type default)
-		)
-	)
-	(wire
-		(pts
 			(xy 340.36 76.2) (xy 340.36 88.9)
 		)
@@
 	(wire
 		(pts
+			(xy 311.15 31.75) (xy 335.28 31.75)
+		)
+		(stroke
+			(width 0)
+			(type default)
+		)
+	)
+	(wire
+		(pts
 			(xy 90.17 181.61) (xy 95.25 181.61)
 		)
@@
 	(wire
 		(pts
-			(xy 311.15 31.75) (xy 311.15 109.22)
+			(xy 311.15 31.75) (xy 311.15 38.1)
 		)
 		(stroke
@@
 	(wire
 		(pts
+			(xy 311.15 48.26) (xy 311.15 109.22)
+		)
+		(stroke
+			(width 0)
+			(type default)
+		)
+	)
+	(wire
+		(pts
 			(xy 113.03 167.64) (xy 125.73 167.64)
 		)
@@
 			"AAAAAAAAAAAAAAAAAAAAAAAAAAAAAAAAAAAAAAAAAAAAAACRRnmGAHIBgAAAAAAAAAAAAAAAAAAA"
 			"AAAAAAAAAAAAAJdGe4YAhwCAAAAAAAAAAAAAAAAAAAAAAAAAAAAAAAAAlUZ9hgBzAYAAAAAAAAAA"
-			"AAAAAAAAAAAAAAAAAAAAAAAAAAAAAAAAAAAAAAAAAAAAAAAAAAAAAAAAAAAAAAAAAGlGcYYAdA=="
+			"AAAAAAAAAAAAAAAAAAAAAAAAAAAAAAAAAAAAAAAAAAAAAAAAAAAAAAAAAAAAAAAAAGlGcYYAdAAA"
+			"AAAAAAAAAAAAAAAAAAAAAAAAAAAAAAAAAAAAAAAAAAAAAAAAAAAAAAAAAAAAAAAAAAAAAAAAAAAA"
+			"AAAAAAAAAAAAAAAAAAAAAAAAAAAAAAAAAAAAAAAAAAAAAAAAAAAAAAAAAAAAAAAAAAAAAAAAAAAA"
+			"AAAAAAAAAAAAAAAAAAAAAAAAAAAAAAAAAAAAAAAAAAAAAAAAAAAAAAAAAAAAAAAAAAAAAAAAAAAA"
+			"AAAAAAAAAAAAAAAAAAAAAAAAAAAAAAAAAAAAAAAAAAAAAAAAAAAAAAAAAAAAAAAAAAAAAAAAAAAA"
+			"AAAAAAAAAAAAAAAAAAAAAAAAAAAAAAAAAAAAAAAAAAAAAAAAAAAAAAAAAAAAAAAAAAAAAAAAAAAA"
+			"AAAAAAAAAAAAAAAAAAAAAAAAAAAAAAAAAAAAAAAAAAAAAAAAAAAAAAAAAAAAAAAAAAAAAAAAAAAA"
+			"AAAAAAAAAAAAAAAAAAAAAAAAAAAAAAAAAAAAAAAAAAAAAAAAAAAAAAAAAAAAAAAAAAAAAAAAAAAA"
+			"AAAAAAAAAAAAAAAAAAAAAAAAAAAAAAAAAAAAAAAAAAAAAAAAAAAAAAAAAAAAAAAAAAAAAAAAAAAA"
+			"AAAAAAAAAAAAAAAAAAAAAAAAAAAAAAAAAAAAAAAAAAAAAAAAAAAAAAAAAAAAAAAAAAAAAAAAAAAA"
+			"AAAAAAAAAAAAAAAAAAAAAAAAAAAAAAAAAAAAAAAAAAAAAAAAAAAAAAAAAAAAAAAAAAAAAAAAAAAA"
+			"AAAAAAAAAAAAAAAAAAAAAAAAAAAAAAAAAAAAAAAAAAAAAAAAAAAAAAAAAAAAAAAAAAAAAAAAAAAA"
+			"AAAAAAAAAAAAAAAAAAAAAAAAAAAAAAAAAAAAAAAAAAAAAAAAAAAAAAAAAAAAAAAAAAAAAAAAAAAA"
+			"AAAAAAAAAAAAAAAAAAAAAAAAAAAAAAAAAAAAAAAAAAAAAAAAAAAAAAAAAAAAAAAAAAAAAAAAAAAA"
+			"AAAAAAAAAAAAAAAAAAAAAAAAAAAAAAAAAAAAAAAAAAAAAAAAAAAAAAAAAAAAAAAAAAAAAAAAAAAA"
+			"AAAAAAAAAAAAAAAAAAAAAAAAAAAAAAAAAAAAAAAAAAAAAAAAAAAAAAAAAAAAAAAAAAAAAAAAAAAA"
+			"AAAAAAAAAAAAAAAAAAAAAAAAAAAAAAAAAAAAAAAAAAAAAAAAAAAAAAAAAAAAAAAAAAAAAAAAAAAA"
+			"AAAAAAAAAAAAAAAAAAAAAAAAAAAAAAAAAAAAAAAAAAAAAAAAAAAAAAAAAAAAAAAAAAAAAAAAAAAA"
+			"AAAAAAAAAAAAAAAAAAAAAAAAAAAAAAAAAAAAAAAAAAAAAAAAAAAAAAAAAAAAAAAAAAAAAAAAAA=="
 		)
 	)
 	(image
-		(at 340.36 212.09)
-		(scale 0.45279)
+		(at 342.9 177.8)
+		(scale 0.299693)
 		(data "/9j/4AAQSkZJRgABAQEASABIAAD/2wBDAAEBAQEBAQEBAQEBAQEBAQEBAQEBAQEBAQEBAQEBAQEB"
 			"AQEBAQICAQECAQEBAgICAgICAgICAQICAgICAgICAgL/2wBDAQEBAQEBAQEBAQECAQEBAgICAgIC"
@@
 			"AAAAAAAAAAAAAAAAAAAAAAAAAAAAAAAAAAAAAAAAAAAAAAAAAAAAAAAAAAAAAAAAAAAAAAAAAAAA"
 			"AAAAAAAAAAAAAAAAAAAAAAAAAAAAAAAAAAAAAAAAAAAAAAAAAAAAAAAAAAAAAAAAAAAAAAAAAGil"
-			"HJIAswCAAAAAAAAAAAAAAAAAAAAAAAA="
+			"HJIAswCAAAAAAAAAAAAAAAAAAAAAAAAAAAAAAAAAAAAAAAAAAAAAAAAAAAAAAAAAAAAAAAAAAAAA"
+			"AAAAAAAAAAAAAAAAAAAAAAAAAAAAAAAAAAAAAAAAAAAAAAAAAAAAAAAAAAAAAAAAAAAAAAAAAAAA"
+			"AAAAAAAAAAAAAAAAAAAAAAAAAAAAAAAAAAAAAAAAAAAAAAAAAAAAAAAAAAAAAAAAAAAAAAAAAAAA"
+			"AAAAAAAAAAAAAAAAAAAAAAAAAAAAAAAAAAAAAAAAAAAAAAAAAAAAAAAAAAAAAAAAAAAAAAAAAAAA"
+			"AAAAAAAAAAAAAAAAAAAAAAAAAAAAAAAAAAAAAAAAAAAAAAAAAAAAAAAAAAAAAAAAAAAAAAAAAAAA"
+			"AAAAAAAAAAAAAAAAAAAAAAAAAAAAAAAAAAAAAAAAAAAAAAAAAAAAAAAAAAAAAAAAAAAAAAAAAAAA"
+			"AAAAAAAAAAAAAAAAAAAAAAAAAAAAAAAAAAAAAAAAAAAAAAAAAAAAAAAAAAAAAAAAAAAAAAAAAAAA"
+			"AAAAAAAAAAAAAAAAAAAAAAAAAAAAAAAAAAAAAAAAAAAAAAAAAAAAAAAAAAAAAAAAAAAAAAAAAAAA"
+			"AAAAAAAAAAAAAAAAAAAAAAAAAAAAAAAAAAAAAAAAAAAAAAAAAAAAAAAAAAAAAAAAAAAAAAAAAAAA"
+			"AAAAAAAAAAAAAAAAAAAAAAAAAAAAAAAAAAAAAAAAAAAAAAAAAAAAAAAAAAAAAAAAAAAAAAAAAAAA"
+			"AAAAAAAAAAAAAAAAAAAAAAAAAAAAAAAAAAAAAAAAAAAAAAAAAAAAAAAAAAAAAAAAAAAAAAAAAAAA"
+			"AAAAAAAAAAAAAAAAAAAAAAAAAAAAAAAAAAAAAAAAAAAAAAAAAAAAAAAAAAAAAAAAAAAAAAAAAAAA"
+			"AAAAAAAAAAAAAAAAAAAAAAAAAAAAAAAAAAAAAAAAAAAAAAAAAAAAAAAAAAAAAAAAAAAAAAAAAAAA"
+			"AAAAAAAAAAAAAAAAAAAAAAAAAAAAAAAAAAAAAAAAAAAAAAAAAAAAAAAAAAAAAAAAAAAAAAAAAAAA"
+			"AAAAAAAAAAAAAAAAAAAAAAAAAAAAAAAAAAAAAAAAAAAAAAAAAAAAAAAAAAAAAAAAAAAAAAAAAAAA"
+			"AAAAAAAAAAAAAAAAAAAAAAAAAAAAAAAAAAAAAAAAAAAAAAAAAAAAAAAAAAAAAAAAAAAAAAAAAAAA"
+			"AAAAAAAAAAAAAAAAAAAAAAAAAAAAAAAAAAAAAAAAAAAAAAAAAAAAAAAAAAAAAAAAAAAAAAAAAAAA"
+			"AAAAAAAAAAAAAAAAAAAAAAAAAAAAAAAAAAAAAAAAAAAAAAAAAAAAAAAAAAAAAAAAAAAAAAAAAAAA"
+			"AAAAAAAAAAAAAAAAAAAAAAAAAAAAAA=="
 		)
 	)
@@
 	)
 	(label "NO1"
-		(at 328.93 31.75 0)
+		(at 313.69 31.75 0)
 		(effects
 			(font
@@
 					(unit 1)
 				)
+			)
+		)
+	)
+	(symbol
+		(lib_id "Switch:SW_DPST_x2")
+		(at 311.15 43.18 90)
+		(unit 1)
+		(exclude_from_sim no)
+		(in_bom yes)
+		(on_board yes)
+		(dnp no)
+		(fields_autoplaced yes)
+		(property "Reference" "SW1"
+			(at 312.42 41.9099 90)
+			(effects
+				(font
+					(size 1.27 1.27)
+				)
+				(justify right)
+			)
+		)
+		(property "Value" "DISABILITA"
+			(at 312.42 44.4499 90)
+			(effects
+				(font
+					(size 1.27 1.27)
+				)
+				(justify right)
+			)
+		)
+		(property "Footprint" ""
+			(at 311.15 43.18 0)
+			(effects
+				(font
+					(size 1.27 1.27)
+				)
+				(hide yes)
+			)
+		)
+		(property "Datasheet" "~"
+			(at 311.15 43.18 0)
+			(effects
+				(font
+					(size 1.27 1.27)
+				)
+				(hide yes)
+			)
+		)
+		(property "Description" "Single Pole Single Throw (SPST) switch, separate symbol"
+			(at 311.15 43.18 0)
+			(effects
+				(font
+					(size 1.27 1.27)
+				)
+				(hide yes)
+			)
+		)
+		(pin "1"
+		)
+		(pin "2"
+		)
+		(pin "3"
+		)
+		(pin "4"
+		)
+		(instances
+			(project ""
+				(path "/f628e06f-c79c-4595-aa2f-837938629d9e"
+					(reference "SW1")
+					(unit 1)
+				)

Commit message: 5/6
Parts:
- removed K4: N.M., Relay_THT:Relay_SPDT_HsinDa_Y14, symbol Relay:Y14x-1C-xxDS
- added D-OPZIONALE: 1N4001, Diode_THT:D_DO-41_SOD81_P10.16mm_Horizontal, symbol Diode:1N4001
- added J10, J11, J6, J7, J8, J9: Conn_01x01_Pin, symbol Connector:Conn_01x01_Pin
- added R23: 10ohm 5watt, Resistor_THT:R_Axial_DIN0204_L3.6mm_D1.6mm_P2.54mm_Vertical, symbol Device:R_Small
- added SW2: DISABILITA BLUETOOTH, symbol Switch:SW_DPST_x2
- SW1: value DISABILITA -> DISABILITA MANT.
Connections:
- net +5V: now also SW2.1 (A), SW2.2 (B)
- net +CARICA SOLARE: now also BT1.1 (+)
- net NO1: no longer SW1.2 (B)
- net at BT2.1 (+): now also D-OPZIONALE.1 (K)
- net at BT1.2 (-), BT2.2 (-): now also J6.1 (Pin_1), J8.1 (Pin_1)
- new net: J7.1 (Pin_1), SW1.2 (B)
- new net: D-OPZIONALE.2 (A), J11.1 (Pin_1), R23.1
- new net: J10.1 (Pin_1), J9.1 (Pin_1), R23.2
Other:
- note added: "10V=1AMP"
- note added: "D2 e D4 SOSTITUIRE CON JUMPER 2 PIN"
- note added: "PRINCIPALE"
- note added: "SECONDARIO"
- note added: "SEMAF GIALLO"
- note added: "SEMAF ROSSO"
- note added: "SEMAF VERDE"
- note removed: "30"
- note removed: "85"
- note removed: "86"
- note removed: "87"
- note removed: "87A"
- note removed: "BLU"
- note removed: "GIALLO"
- note removed: "VERDE"
- moved on the sheet: SW1A
