File: Kicad/Camper_Energy_Saver_Wiring.kicad_sch (KiCad schematic)
At the start: 7 parts, among them J10 Conn_01x01_Pin, J11 Conn_01x01_Pin, J12 Conn_01x01_Pin, J13 Conn_01x01_Pin, SW1 DISABILITA MANT.

Commit message: Update wiring schematic and add images
Changed schematic paper size to A4, added a large arrow symbol, updated component positions, text labels, and wiring coordinates in the KiCad schematic. Added two new image files: 'mammu4t.png' and 'wiring schematic.jpg'.
Parts:
- added J14, J15, J16, J17, J18, J19, J20, J21, J22, J23, J24, J25, J26, J27, J28, J29, J30, J31, J32, J33, J34: Conn_01x01_Pin, symbol Connector:Conn_01x01_Pin
Connections:
- net +CARICA SOLARE: now also J22.1 (Pin_1)
- net GNDREF: now also J27.1 (Pin_1), J28.1 (Pin_1), J30.1 (Pin_1)
- net at SW1.1 (A): now also J31.1 (Pin_1), J33.1 (Pin_1)
- net at J11.1 (Pin_1), SW1.2 (B): now also J26.1 (Pin_1)
- net at BT2.1 (+): now also J25.1 (Pin_1)
- net at BT1.2 (-), BT2.2 (-): now also J23.1 (Pin_1), J24.1 (Pin_1)
- net at J10.1 (Pin_1): now also J34.1 (Pin_1)
- net at J13.1 (Pin_1): now also J14.1 (Pin_1)
- new net: J17.1 (Pin_1), J29.1 (Pin_1), J32.1 (Pin_1)
- new net: J15.1 (Pin_1), J16.1 (Pin_1)
Other:
- moved on the sheet: BT1, BT2, SW1A
